File: Synchronous Rectifier.kicad_sch (KiCad schematic)
At the start: 145 parts, among them IC2 LM2776DBVR, IC3 ADA4817-1ARDZ-R7, J1 Conn_Coaxial, P1 Conn_Plug_2P, P2 Conn_Plug_2P, P3 Conn_Plug_2P, P4 Conn_Plug_2P, Q1 IGB110S10S1, Q2 IGB110S10S1, Q3 IGB110S10S1, Q4 IGB110S10S1, U1 LMG1210RVRR, U10 74AHCT1G86, U11 74AHCT1G86, U13 TLV3601DBVR, U2 TLV3601DBVR, U3 TLV3601DBVR, U6 74LVC1G17, U9 LMG1210RVRR

Commit message: first round changes, before ltspice
Parts:
- removed C16, C42, C43, C57, C60: 1u, Capacitor_SMD:C_0603_1608Metric, symbol Device:C
- removed C26: 10u, Capacitor_SMD:C_0603_1608Metric, symbol Device:C
- removed C41: 100n, Capacitor_SMD:C_0603_1608Metric, symbol Device:C
- removed C44: 10n, Capacitor_SMD:C_0603_1608Metric, symbol Device:C
- removed D6: BAT46W, Diode_SMD:D_SOD-123F, symbol Diode:1N5819WS
- removed J1: Conn_Coaxial, Connector_Coaxial:SMA_Amphenol_132134_Vertical, symbol Connector:Conn_Coaxial
- removed P1, P2, P3, P4: Conn_Plug_2P, bananaPlug:571-0500, symbol Connector:Conn_Plug_2P
- removed Q1, Q2, Q3, Q4: IGB110S10S1, GaN:IFX-PG-TSON-4-2-V, symbol GaNFET:IGB110S101
- removed R13: 1k, Resistor_SMD:R_0603_1608Metric, symbol Device:R_US
- removed R21: 100, Resistor_SMD:R_0603_1608Metric, symbol Device:R_US
- removed R31: 100k, Resistor_SMD:R_0603_1608Metric, symbol Device:R_US
- removed R36: 470, Resistor_SMD:R_0603_1608Metric, symbol Device:R_US
- removed R53, R54: 4.7k, Resistor_SMD:R_0603_1608Metric, symbol Device:R_US
- removed S2: G13AP, G13AP:G13AP, symbol G13AP:G13AP
- removed TP31, TP32: tp, TestPoint:TestPoint_THTPad_D2.0mm_Drill1.0mm, symbol Connector:TestPoint
- removed U13: TLV3601DBVR, Package_TO_SOT_SMD:TSOT-23-5_HandSoldering, symbol tlv3601:TLV3601DBVR
- removed U6: 74LVC1G17, Package_TO_SOT_SMD:SOT-23-5_HandSoldering, symbol 74xGxx:74LVC1G17
- added BT1: BC4AAB, BC4AAB:BAT_BC4AAB, symbol BC4AAB:BC4AAB
- added Q1, Q2, Q3, Q4: BSC105N15LS5, BSC105N15LS5:IFX-PG-TDSON-8-66-V, symbol BSC105N15LS5:BSC105N15LS5
- added ReceiverCoil1: Screw_Terminal_01x02, TestPoint:TestPoint_Keystone_5010-5014_Multipurpose, symbol Connector:Screw_Terminal_01x02
- C1, C58: value 250p -> 33n
- C11: value 10n -> 100n
- C14: value 51p -> 2.7n
- C15: value 10n -> 180n
- C4, C5: value 80p -> 68p
- C47: value 660p -> 1u
- R12: value 1k -> 10k
- R18: value 32.4k -> 33.2k
- R19: value 6.65k -> 6.81k
- R2, R3, R37, R4, R5, R6: value 4.7k -> 22k
- R20, R22: value 1k -> 3.3k
- R45, R46: value 14.7k -> 470k
Connections:
- net 5V: now also C11.2, R12.2, TP6.1, U3.3 (IN+), BT1.+
- net G1: now also Q1.4 (GATE)
- net G2: now also Q3.4 (GATE)
- net G3: now also Q2.4 (GATE)
- net G4: now also Q4.4 (GATE)
- net GND: now also BT1.-, Q2.1 (SOURCE_1), Q2.2 (SOURCE_2), Q2.3 (SOURCE_3), Q4.1 (SOURCE_1), Q4.2 (SOURCE_2), Q4.3 (SOURCE_3)
- net Is-: now also ReceiverCoil1.1 (Pin_1)
- net Out+: now also Q1.5 (DRAIN_1), Q1.6 (DRAIN_2), Q1.7 (DRAIN_3), Q1.8 (DRAIN_4), Q3.5 (DRAIN_1), Q3.6 (DRAIN_2), Q3.7 (DRAIN_3), Q3.8 (DRAIN_4)
- net S1: now also Q1.1 (SOURCE_1), Q1.2 (SOURCE_2), Q1.3 (SOURCE_3), Q2.5 (DRAIN_1), Q2.6 (DRAIN_2), Q2.7 (DRAIN_3), Q2.8 (DRAIN_4)
- net S2: now also Q3.1 (SOURCE_1), Q3.2 (SOURCE_2), Q3.3 (SOURCE_3), Q4.5 (DRAIN_1), Q4.6 (DRAIN_2), Q4.7 (DRAIN_3), Q4.8 (DRAIN_4)
- net L-: no longer names the net of C58.1
- net L-: now also ReceiverCoil1.2 (Pin_2)
Other:
- note removed: "Banana Connectors"
- note removed: "Start-up and Control Logic"
- moved on the sheet: C7, C8, R10, R7, R9, U1

Commit message: setup 2 ltspice, need to update resistors based on graphs
Parts:
- added C9: C, Package_QFP:TQFP-44_10x10mm_P0.8mm, symbol Device:C
- added R8: 10k, Resistor_THT:R_Array_SIP4, symbol Device:R_US
Connections:
- net 5V: now also R8.1; no longer C11.2, R12.2, TP6.1, U3.3 (IN+)
- net FB: now also C9.1
- net GND: now also C9.2
- new net: C11.2, R12.2, R8.2, TP6.1, U3.3 (IN+)
